Commit message: update camera

File: kubot_description/urdf/camera_xacro/d435i.urdf.xacro (robot description, xacro)
@@ -9,5 +9,5 @@
 				<origin xyz="0 0 0" rpy="0 0 0" />
 				<geometry>
-					<mesh filename="package://kubot_description/meshes/camera_frame/d435i/camera_link.stl" scale="0.001 0.001 0.001" />
+					<mesh filename="package://kubot_description/meshes/camera_frame/$(arg camera)/camera_link.stl" scale="0.001 0.001 0.001" />
 				</geometry>
 				<xacro:material_dark_grey />
@@ -16,5 +16,5 @@
 				<origin xyz="0 0 0" rpy="0 0 0" />
 				<geometry>
-					<mesh filename="package://kubot_description/meshes/camera_frame/d435i/camera_link.stl" scale="0.001 0.001 0.001" />
+					<mesh filename="package://kubot_description/meshes/camera_frame/$(arg camera)/camera_link.stl" scale="0.001 0.001 0.001" />
 				</geometry>
 				<xacro:material_white />

File: kubot_description/urdf/camera_xacro/logi-c615.urdf.xacro (robot description, xacro)
@@ -9,5 +9,5 @@
 				<origin xyz="0 0 0" rpy="0 0 0" />
 				<geometry>
-					<mesh filename="package://kubot_description/meshes/camera_frame/$(arg sensor)/camera_link.stl" />
+					<mesh filename="package://kubot_description/meshes/camera_frame/$(arg camera)/camera_link.stl" />
 				</geometry>
 				<xacro:material_dark_grey />
@@ -16,5 +16,5 @@
 				<origin xyz="0 0 0" rpy="0 0 0" />
 				<geometry>
-					<mesh filename="package://kubot_description/meshes/camera_frame/$(arg sensor)/camera_link.stl" />
+					<mesh filename="package://kubot_description/meshes/camera_frame/$(arg camera)/camera_link.stl" />
 				</geometry>
 				<xacro:material_white />

File: kubot_description/urdf/kubot.urdf.xacro (robot description, xacro)
@@ -3,5 +3,5 @@
 	<xacro:arg name="model" default="" />
 	<xacro:arg name="lidar" default="" />
-	<xacro:arg name="sensor" default="" />
+	<xacro:arg name="camera" default="" />
 	<!-- Robot in the ground -->
 	<xacro:macro name="kubot_robot">
@@ -20,5 +20,5 @@
 		<xacro:lidar lidar_joint_xyz="${lidar_joint_xyz}" lidar_joint_rpy="${lidar_joint_rpy}"></xacro:lidar>
 		<!-- Camera Frame -->
-		<xacro:include filename="$(find kubot_description)/urdf/camera_xacro/$(arg sensor).urdf.xacro" />
+		<xacro:include filename="$(find kubot_description)/urdf/camera_xacro/$(arg camera).urdf.xacro" />
 		<xacro:camera_sensor camera_joint_xyz="${camera_joint_xyz}" camera_joint_rpy="${camera_joint_rpy}"></xacro:camera_sensor>
 	</xacro:macro>
